Commit message: Craig drives in Gazebo: physics body + diff-drive plugin

File: urdf/my_robot.urdf (robot description, URDF)
Before this commit: robot craig, 4 links, 3 joints
Links:
- link base_link: mass None -> 1.0; geometry collision box size=0.3 0.2 0.1; visual box size=0.3 0.2 0.1
- link caster: mass None -> 0.05; geometry collision sphere radius=0.03; visual sphere radius=0.03
- link left_wheel: mass None -> 0.1; geometry collision cylinder length=0.04 radius=0.05; visual cylinder length=0.04 radius=0.05
- link right_wheel: mass None -> 0.1; geometry collision cylinder length=0.04 radius=0.05; visual cylinder length=0.04 radius=0.05

Commit message: Full sim bringup: launch file + lidar in RViz, auto-loaded config

File: urdf/my_robot.urdf (robot description, URDF)
Before this commit: robot craig, 4 links, 3 joints
Links:
- added link lidar_link, mass 0.05; collision cylinder length=0.02 radius=0.035; visual cylinder length=0.02 radius=0.035
Joints:
- added joint lidar_joint: type fixed, parent base_link, child lidar_link, origin xyz=0 0 0.06 rpy=0 0 0
