Commit message: Daily build log update

File: urdf/balancer.urdf (robot description, URDF)
Before this commit: robot craig2, 4 links, 3 joints
Links:
- added link lidar_link, mass 0.12; collision cylinder length=0.02 radius=0.035; visual cylinder length=0.02 radius=0.035
Joints:
- added joint lidar_joint: type fixed, parent base_link, child lidar_link, origin xyz=0 0 0.42 rpy=0 0 0
